Commit message: add p3d ground truth; tabs to spaces

File: urdf/kobuki_gazebo.urdf.xacro (robot description, xacro)
@@ -2,140 +2,140 @@
 <robot name="kobuki_sim" xmlns:xacro="http://ros.org/wiki/xacro">
   <xacro:macro name="kobuki_sim">
-	  <gazebo reference="wheel_left_link">
-	    <mu1>1.0</mu1>
-	    <mu2>1.0</mu2>
-	    <kp>1000000.0</kp>
-	    <kd>100.0</kd>
-	    <minDepth>0.001</minDepth>
-	    <maxVel>1.0</maxVel>
-	  </gazebo>
-	  <gazebo reference="wheel_right_link">
-	    <mu1>1.0</mu1>
-	    <mu2>1.0</mu2>
-	    <kp>1000000.0</kp>
-	    <kd>100.0</kd>
-	    <minDepth>0.001</minDepth>
-	    <maxVel>1.0</maxVel>
-	  </gazebo>
-	  <gazebo reference="caster_front_link">
-	    <mu1>0.0</mu1>
-	    <mu2>0.0</mu2>
-	    <kp>1000000.0</kp>
-	    <kd>100.0</kd>
-	    <minDepth>0.001</minDepth>
-	    <maxVel>1.0</maxVel>
-	  </gazebo>
-	  <gazebo reference="caster_back_link">
-	    <mu1>0.0</mu1>
-	    <mu2>0.0</mu2>
-	    <kp>1000000.0</kp>
-	    <kd>100.0</kd>
-	    <minDepth>0.001</minDepth>
-	    <maxVel>1.0</maxVel>
-	  </gazebo>
-	  <gazebo reference="base_link">
-	    <mu1>0.3</mu1>
-	    <mu2>0.3</mu2>
-	    <sensor type="contact" name="bumpers">
-	      <always_on>1</always_on>
-	      <update_rate>50.0</update_rate>
-	      <visualize>true</visualize>
-	      <contact>
-	        <collision>base_footprint_fixed_joint_lump__base_collision</collision>
-	      </contact>
-	    </sensor>
-	  </gazebo>
-	  <gazebo reference="cliff_sensor_left_link">
-	    <sensor type="ray" name="cliff_sensor_left">
-	      <always_on>true</always_on>
-	      <update_rate>50</update_rate>
-	      <visualize>true</visualize>
-	      <ray>
-	        <scan>
-	          <horizontal>
-	            <samples>50</samples>
-	            <resolution>1.0</resolution>
-	            <min_angle>-0.0436</min_angle>  <!-- -2.5 degree -->
-	            <max_angle>0.0436</max_angle> <!-- 2.5 degree -->
-	          </horizontal>
-			<!-- Cannot use vertical rays until this bug is resolved -->
-			<!-- https://bitbucket.org/osrf/gazebo/issue/509/vertical-sensor-doesnt-works -->
-			<!-- <vertical> -->
-			<!--     <samples>50</samples> -->
-			<!--     <resolution>1.0</resolution> -->
-			<!--     <min_angle>-0.0436</min_angle>  -2.5 degree -->
-			<!--     <max_angle>0.0436</max_angle> 2.5 degree -->
-			<!-- </vertical> -->
-	        </scan>
-	        <range>
-	          <min>0.01</min>
-	          <max>0.15</max>
-	          <resolution>1.0</resolution>
-	        </range>
-	      </ray>
-	    </sensor>
-	  </gazebo>
-	  <gazebo reference="cliff_sensor_right_link">
-	    <sensor type="ray" name="cliff_sensor_right">
-	      <always_on>true</always_on>
-	      <update_rate>50</update_rate>
-	      <visualize>true</visualize>
-	      <ray>
-	        <scan>
-	          <horizontal>
-	            <samples>50</samples>
-	            <resolution>1.0</resolution>
-	            <min_angle>-0.0436</min_angle>  <!-- -2.5 degree -->
-	            <max_angle>0.0436</max_angle> <!-- 2.5 degree -->
-	          </horizontal>
-			<!-- Cannot use vertical rays until this bug is resolved -->
-			<!-- https://bitbucket.org/osrf/gazebo/issue/509/vertical-sensor-doesnt-works -->
-			<!-- <vertical> -->
-			<!--     <samples>50</samples> -->
-			<!--     <resolution>1.0</resolution> -->
-			<!--     <min_angle>-0.0436</min_angle>  -2.5 degree -->
-			<!--     <max_angle>0.0436</max_angle> 2.5 degree -->
-			<!-- </vertical> -->
-	        </scan>
-	        <range>
-	          <min>0.01</min>
-	          <max>0.15</max>
-	          <resolution>1.0</resolution>
-	        </range>
-	      </ray>
-	    </sensor>
-	  </gazebo>
-	  <gazebo reference="cliff_sensor_front_link">
-	    <sensor type="ray" name="cliff_sensor_front">
-	      <always_on>true</always_on>
-	      <update_rate>50</update_rate>
-	      <visualize>true</visualize>
-	      <ray>
-	        <scan>
-	          <horizontal>
-	            <samples>50</samples>
-	            <resolution>1.0</resolution>
-	            <min_angle>-0.0436</min_angle>  <!-- -2.5 degree -->
-	            <max_angle>0.0436</max_angle> <!-- 2.5 degree -->
-	          </horizontal>
-			<!-- Cannot use vertical rays until this bug is resolved -->
-			<!-- https://bitbucket.org/osrf/gazebo/issue/509/vertical-sensor-doesnt-works -->
-			<!-- <vertical> -->
-			<!--     <samples>50</samples> -->
-			<!--     <resolution>1.0</resolution> -->
-			<!--     <min_angle>-0.0436</min_angle>  -2.5 degree -->
-			<!--     <max_angle>0.0436</max_angle> 2.5 degree -->
-			<!-- </vertical> -->
-	        </scan>
-	        <range>
-	          <min>0.01</min>
-	          <max>0.15</max>
-	          <resolution>1.0</resolution>
-	        </range>
-	      </ray>
-	    </sensor>
-	  </gazebo>
-	  <gazebo reference="gyro_link">
-	   <sensor type="imu" name="imu">
+      <gazebo reference="wheel_left_link">
+        <mu1>1.0</mu1>
+        <mu2>1.0</mu2>
+        <kp>1000000.0</kp>
+        <kd>100.0</kd>
+        <minDepth>0.001</minDepth>
+        <maxVel>1.0</maxVel>
+      </gazebo>
+      <gazebo reference="wheel_right_link">
+        <mu1>1.0</mu1>
+        <mu2>1.0</mu2>
+        <kp>1000000.0</kp>
+        <kd>100.0</kd>
+        <minDepth>0.001</minDepth>
+        <maxVel>1.0</maxVel>
+      </gazebo>
+      <gazebo reference="caster_front_link">
+        <mu1>0.0</mu1>
+        <mu2>0.0</mu2>
+        <kp>1000000.0</kp>
+        <kd>100.0</kd>
+        <minDepth>0.001</minDepth>
+        <maxVel>1.0</maxVel>
+      </gazebo>
+      <gazebo reference="caster_back_link">
+        <mu1>0.0</mu1>
+        <mu2>0.0</mu2>
+        <kp>1000000.0</kp>
+        <kd>100.0</kd>
+        <minDepth>0.001</minDepth>
+        <maxVel>1.0</maxVel>
+      </gazebo>
+      <gazebo reference="base_link">
+        <mu1>0.3</mu1>
+        <mu2>0.3</mu2>
+        <sensor type="contact" name="bumpers">
+          <always_on>1</always_on>
+          <update_rate>50.0</update_rate>
+          <visualize>true</visualize>
+          <contact>
+            <collision>base_footprint_fixed_joint_lump__base_collision</collision>
+          </contact>
+        </sensor>
+      </gazebo>
+      <gazebo reference="cliff_sensor_left_link">
+        <sensor type="ray" name="cliff_sensor_left">
+          <always_on>true</always_on>
+          <update_rate>50</update_rate>
+          <visualize>true</visualize>
+          <ray>
+            <scan>
+              <horizontal>
+                <samples>50</samples>
+                <resolution>1.0</resolution>
+                <min_angle>-0.0436</min_angle>  <!-- -2.5 degree -->
+                <max_angle>0.0436</max_angle> <!-- 2.5 degree -->
+              </horizontal>
+            <!-- Cannot use vertical rays until this bug is resolved -->
+            <!-- https://bitbucket.org/osrf/gazebo/issue/509/vertical-sensor-doesnt-works -->
+            <!-- <vertical> -->
+            <!--     <samples>50</samples> -->
+            <!--     <resolution>1.0</resolution> -->
+            <!--     <min_angle>-0.0436</min_angle>  -2.5 degree -->
+            <!--     <max_angle>0.0436</max_angle> 2.5 degree -->
+            <!-- </vertical> -->
+            </scan>
+            <range>
+              <min>0.01</min>
+              <max>0.15</max>
+              <resolution>1.0</resolution>
+            </range>
+          </ray>
+        </sensor>
+      </gazebo>
+      <gazebo reference="cliff_sensor_right_link">
+        <sensor type="ray" name="cliff_sensor_right">
+          <always_on>true</always_on>
+          <update_rate>50</update_rate>
+          <visualize>true</visualize>
+          <ray>
+            <scan>
+              <horizontal>
+                <samples>50</samples>
+                <resolution>1.0</resolution>
+                <min_angle>-0.0436</min_angle>  <!-- -2.5 degree -->
+                <max_angle>0.0436</max_angle> <!-- 2.5 degree -->
+              </horizontal>
+            <!-- Cannot use vertical rays until this bug is resolved -->
+            <!-- https://bitbucket.org/osrf/gazebo/issue/509/vertical-sensor-doesnt-works -->
+            <!-- <vertical> -->
+            <!--     <samples>50</samples> -->
+            <!--     <resolution>1.0</resolution> -->
+            <!--     <min_angle>-0.0436</min_angle>  -2.5 degree -->
+            <!--     <max_angle>0.0436</max_angle> 2.5 degree -->
+            <!-- </vertical> -->
+            </scan>
+            <range>
+              <min>0.01</min>
+              <max>0.15</max>
+              <resolution>1.0</resolution>
+            </range>
+          </ray>
+        </sensor>
+      </gazebo>
+      <gazebo reference="cliff_sensor_front_link">
+        <sensor type="ray" name="cliff_sensor_front">
+          <always_on>true</always_on>
+          <update_rate>50</update_rate>
+          <visualize>true</visualize>
+          <ray>
+            <scan>
+              <horizontal>
+                <samples>50</samples>
+                <resolution>1.0</resolution>
+                <min_angle>-0.0436</min_angle>  <!-- -2.5 degree -->
+                <max_angle>0.0436</max_angle> <!-- 2.5 degree -->
+              </horizontal>
+            <!-- Cannot use vertical rays until this bug is resolved -->
+            <!-- https://bitbucket.org/osrf/gazebo/issue/509/vertical-sensor-doesnt-works -->
+            <!-- <vertical> -->
+            <!--     <samples>50</samples> -->
+            <!--     <resolution>1.0</resolution> -->
+            <!--     <min_angle>-0.0436</min_angle>  -2.5 degree -->
+            <!--     <max_angle>0.0436</max_angle> 2.5 degree -->
+            <!-- </vertical> -->
+            </scan>
+            <range>
+              <min>0.01</min>
+              <max>0.15</max>
+              <resolution>1.0</resolution>
+            </range>
+          </ray>
+        </sensor>
+      </gazebo>
+      <gazebo reference="gyro_link">
+       <sensor type="imu" name="imu">
         <plugin name="gazebo_ros_imu_controller" filename="libgazebo_ros_imu_sensor.so">
           <ros>
@@ -205,8 +205,8 @@
             </z>
           </linear_acceleration>
-	      </imu>
+          </imu>
       </sensor>
-	  </gazebo>
-	  <gazebo>
+      </gazebo>
+      <gazebo>
       <plugin name="differential_drive_controller" filename="libgazebo_ros_diff_drive.so">
         <update_rate>50</update_rate>
@@ -225,5 +225,16 @@
         <odometry_frame>odom</odometry_frame>
         <robot_base_frame>base_footprint</robot_base_frame>
-	    </plugin>
+        </plugin>
+        <!-- publish ground truth -->
+        <plugin name="p3d_ground_truth" filename="libgazebo_ros_p3d.so">
+            <always_on>true</always_on>
+            <update_rate>50.0</update_rate>
+            <body_name>base_footprint</body_name>
+            <topic_name>ground_truth</topic_name>
+            <gaussian_noise>0.001</gaussian_noise>
+            <frame_name>world</frame_name>
+            <xyz_offset>0 0 0</xyz_offset>
+            <rpy_offset>0 0 0</rpy_offset>
+        </plugin>
       <plugin name="kobuki_joint_state" filename="libgazebo_ros_joint_state_publisher.so">
         <ros>
@@ -234,5 +245,5 @@
         <joint_name>wheel_right_joint</joint_name>
       </plugin>
-	  </gazebo>
+      </gazebo>
   </xacro:macro>
 </robot>
