Commit message: Update for ROS 2 Jazzy and GazeboSim Harmonic

File: urdf/kobuki.urdf.xacro (robot description, xacro)
@@ -30,5 +30,5 @@
         <geometry>
           <!-- new mesh -->
-          <mesh filename="package://chris_ros_turtlebot2/models/meshes/main_body.dae" />
+          <mesh filename="file://$(find chris_ros_turtlebot2)/models/meshes/main_body.dae" />
         </geometry>
         <origin xyz="0.001 0 0.05199" rpy="0 0 0"/>
@@ -65,5 +65,5 @@
       <visual>
         <geometry>
-          <mesh filename="package://chris_ros_turtlebot2/models/meshes/wheel.dae"/>
+          <mesh filename="file://$(find chris_ros_turtlebot2)/models/meshes/wheel.dae"/>
         </geometry>
         <origin xyz="0 0 0" rpy="0 0 0"/>
@@ -92,5 +92,5 @@
       <visual>
         <geometry>
-          <mesh filename="package://chris_ros_turtlebot2/models/meshes/wheel.dae"/>
+          <mesh filename="file://$(find chris_ros_turtlebot2)/models/meshes/wheel.dae"/>
         </geometry>
         <origin xyz="0 0 0" rpy="0 0 0"/>

File: urdf/kobuki_gazebo.urdf.xacro (robot description, xacro)
@@ -47,5 +47,5 @@
       </gazebo>
       <gazebo reference="cliff_sensor_left_link">
-        <sensor type="ray" name="cliff_sensor_left">
+        <sensor type="gpu_lidar" name="cliff_sensor_left">
           <always_on>true</always_on>
           <update_rate>50</update_rate>
@@ -59,17 +59,15 @@
                 <max_angle>0.0436</max_angle> <!-- 2.5 degree -->
               </horizontal>
-            <!-- Cannot use vertical rays until this bug is resolved -->
-            <!-- https://bitbucket.org/osrf/gazebo/issue/509/vertical-sensor-doesnt-works -->
-            <!-- <vertical> -->
-            <!--     <samples>50</samples> -->
-            <!--     <resolution>1.0</resolution> -->
-            <!--     <min_angle>-0.0436</min_angle>  -2.5 degree -->
-            <!--     <max_angle>0.0436</max_angle> 2.5 degree -->
-            <!-- </vertical> -->
-            </scan>
+              <vertical>
+                <samples>1</samples>
+                <resolution>1</resolution>
+                <min_angle>0</min_angle>
+                <max_angle>0</max_angle>
+              </vertical>
+          </scan>
             <range>
               <min>0.01</min>
               <max>0.15</max>
-              <resolution>1.0</resolution>
+              <resolution>0.01</resolution>
             </range>
           </ray>
@@ -89,17 +87,15 @@
                 <max_angle>0.0436</max_angle> <!-- 2.5 degree -->
               </horizontal>
-            <!-- Cannot use vertical rays until this bug is resolved -->
-            <!-- https://bitbucket.org/osrf/gazebo/issue/509/vertical-sensor-doesnt-works -->
-            <!-- <vertical> -->
-            <!--     <samples>50</samples> -->
-            <!--     <resolution>1.0</resolution> -->
-            <!--     <min_angle>-0.0436</min_angle>  -2.5 degree -->
-            <!--     <max_angle>0.0436</max_angle> 2.5 degree -->
-            <!-- </vertical> -->
+              <vertical>
+                <samples>1</samples>
+                <resolution>1</resolution>
+                <min_angle>0</min_angle>
+                <max_angle>0</max_angle>
+              </vertical>
             </scan>
             <range>
               <min>0.01</min>
               <max>0.15</max>
-              <resolution>1.0</resolution>
+              <resolution>0.01</resolution>
             </range>
           </ray>
@@ -119,17 +115,15 @@
                 <max_angle>0.0436</max_angle> <!-- 2.5 degree -->
               </horizontal>
-            <!-- Cannot use vertical rays until this bug is resolved -->
-            <!-- https://bitbucket.org/osrf/gazebo/issue/509/vertical-sensor-doesnt-works -->
-            <!-- <vertical> -->
-            <!--     <samples>50</samples> -->
-            <!--     <resolution>1.0</resolution> -->
-            <!--     <min_angle>-0.0436</min_angle>  -2.5 degree -->
-            <!--     <max_angle>0.0436</max_angle> 2.5 degree -->
-            <!-- </vertical> -->
+              <vertical>
+                <samples>1</samples>
+                <resolution>1</resolution>
+                <min_angle>0</min_angle>
+                <max_angle>0</max_angle>
+              </vertical>
             </scan>
             <range>
               <min>0.01</min>
               <max>0.15</max>
-              <resolution>1.0</resolution>
+              <resolution>0.01</resolution>
             </range>
           </ray>
@@ -138,19 +132,8 @@
       <gazebo reference="gyro_link">
        <sensor type="imu" name="imu">
-        <plugin name="gazebo_ros_imu_controller" filename="libgazebo_ros_imu_sensor.so">
-          <ros>
-            <argument>--ros-args</argument>
-            <argument>-r</argument>
-            <argument>~/out:=imu</argument>
-          </ros>
-          <output_type>sensor_msgs/msg/Imu</output_type>
-          <body_name>gyro_link</body_name>
-          <frame_name>gyro_link</frame_name>
-        </plugin>
         <always_on>true</always_on>
         <update_rate>50</update_rate>
         <visualize>false</visualize>
         <imu>
-          <!-- based on original and https://github.com/ros-simulation/gazebo_ros_pkgs/files/2298904/gazebo_ros_imu_sensor.world.txt -->
           <angular_velocity>
             <x>
@@ -160,4 +143,7 @@
                 <bias_mean>0.0000075</bias_mean>
                 <bias_stddev>0.0000008</bias_stddev>
+                <dynamic_bias_stddev>0.00002</dynamic_bias_stddev>
+                <dynamic_bias_correlation_time>400.0</dynamic_bias_correlation_time>
+                <precision>0.00025</precision>
               </noise>
             </x>
@@ -168,4 +154,7 @@
                 <bias_mean>0.0000075</bias_mean>
                 <bias_stddev>0.0000008</bias_stddev>
+                <dynamic_bias_stddev>0.00002</dynamic_bias_stddev>
+                <dynamic_bias_correlation_time>400.0</dynamic_bias_correlation_time>
+                <precision>0.00025</precision>
               </noise>
             </y>
@@ -176,4 +165,7 @@
                 <bias_mean>0.0000075</bias_mean>
                 <bias_stddev>0.0000008</bias_stddev>
+                <dynamic_bias_stddev>0.00002</dynamic_bias_stddev>
+                <dynamic_bias_correlation_time>400.0</dynamic_bias_correlation_time>
+                <precision>0.00025</precision>
               </noise>
             </z>
@@ -194,4 +186,7 @@
                 <bias_mean>0.1</bias_mean>
                 <bias_stddev>0.001</bias_stddev>
+                <dynamic_bias_stddev>0.00002</dynamic_bias_stddev>
+                <dynamic_bias_correlation_time>400.0</dynamic_bias_correlation_time>
+                <precision>0.00025</precision>
               </noise>
             </y>
@@ -202,4 +197,7 @@
                 <bias_mean>0.1</bias_mean>
                 <bias_stddev>0.001</bias_stddev>
+                <dynamic_bias_stddev>0.00002</dynamic_bias_stddev>
+                <dynamic_bias_correlation_time>400.0</dynamic_bias_correlation_time>
+                <precision>0.00025</precision>
               </noise>
             </z>
@@ -209,4 +207,12 @@
       </gazebo>
       <gazebo>
+        <plugin
+          filename="gz-sim-odometry-publisher-system"
+          name="gz::sim::systems::OdometryPublisher">
+          <odom_frame>odom</odom_frame>
+          <robot_base_frame>base_footprint</robot_base_frame>
+        </plugin>
+      </gazebo>
+      <!--gazebo>
       <plugin name="differential_drive_controller" filename="libgazebo_ros_diff_drive.so">
         <update_rate>50</update_rate>
@@ -218,5 +224,5 @@
         <max_wheel_acceleration>1.0</max_wheel_acceleration>
         <command_topic>cmd_vel</command_topic>
-        <!-- output -->
+        <!- - output - ->
         <publish_odom>true</publish_odom>
         <publish_odom_tf>true</publish_odom_tf>
@@ -226,5 +232,5 @@
         <robot_base_frame>base_footprint</robot_base_frame>
         </plugin>
-        <!-- publish ground truth -->
+        <!- - publish ground truth - ->
         <plugin name="p3d_ground_truth" filename="libgazebo_ros_p3d.so">
             <always_on>true</always_on>
@@ -236,5 +242,5 @@
             <rpy_offset>0 0 0</rpy_offset>
             <ros>
-              <!--https://github.com/ros-simulation/gazebo_ros_pkgs/issues/1318-->
+              <!- -https://github.com/ros-simulation/gazebo_ros_pkgs/issues/1318- ->
               <remapping>odom:=ground_truth</remapping>
             </ros>
@@ -248,5 +254,5 @@
         <joint_name>wheel_right_joint</joint_name>
       </plugin>
-      </gazebo>
+      </gazebo -->
   </xacro:macro>
 </robot>

File: urdf/sensors/hokuyo_urg04.urdf.xacro (robot description, xacro)
@@ -1,6 +1,7 @@
 <?xml version="1.0"?>
 <!-- Hokoyu URG-04 lidar model (Simple) -->
-<xacro:robot name="hokuyo_urg04" xmlns:xacro="http://ros.org/wiki/xacro">
-  <xacro:macro name="hokuyo_urg04" params="lidar_name">
+<robot name="hokuyo_urg04" xmlns:xacro="http://www.ros.org/wiki/xacro">
+<xacro:macro name="hokuyo_urg04"
+        params="lidar_name lidar_type sim_gazebo:=^|false visualize_lidar:=^|true">
   <!-- Constants for robot dimensions -->
   <xacro:property name="PI" value="3.1415926535897931"/>
@@ -14,6 +15,4 @@
   <!-- Import Rviz colors -->
   <xacro:include filename="$(find chris_ros_turtlebot2)/urdf/common_properties.urdf.xacro" />
-  <!-- Import all Gazebo-customization elements, including Gazebo colors -->
-  <xacro:include filename="$(find chris_ros_turtlebot2)/urdf/sensors/hokuyo_urg04_gazebo.urdf.xacro" />
   <!-- Hokuyo Laser -->
   <link name="${lidar_name}_base_link">
@@ -27,5 +26,5 @@
       <origin xyz="0 0 0.0175" rpy="0 0 0"/>
       <geometry>
-            <mesh filename="package://chris_ros_turtlebot2/models/meshes/sensors/hokuyo.dae"/>
+            <mesh filename="file://$(find chris_ros_turtlebot2)/models/meshes/sensors/hokuyo.dae"/>
       </geometry>
     </visual>
@@ -51,6 +50,48 @@
     </collision>
   </link>
-  <!-- Simulation sensors -->
-  <xacro:hokuyo_urg04_sim/>
-  </xacro:macro>
-</xacro:robot>
+  <xacro:if value="${sim_gazebo}">
+    <!-- Simulation sensors -->
+    <gazebo reference="${lidar_name}_base_link">
+      <preserveFixedJoint>true</preserveFixedJoint>
+    </gazebo>
+    <gazebo reference="${lidar_name}_laser">
+      <preserveFixedJoint>true</preserveFixedJoint>
+    </gazebo>
+    <gazebo reference="${lidar_name}_laser">
+      <material>Gazebo/Grey</material>
+      <sensor name="${lidar_name}_sensor" type="${lidar_type}" >
+          <topic>${lidar_name}_node/scan_raw</topic>
+          <pose relative_to='${lidar_name}_laser'>0 0 0 0 0 0</pose>
+          <visualize>${visualize_lidar}</visualize>
+          <update_rate>30</update_rate>
+          <always_on>1</always_on>
+          <gz_frame_id>${lidar_name}_laser</gz_frame_id>
+          <ray>
+            <scan>
+              <horizontal>
+                <samples>682</samples>
+                <resolution>1</resolution>
+                <min_angle>-${PI*2.0/3.0}</min_angle>
+                <max_angle> ${PI*2.0/3.0}</max_angle>
+              </horizontal>
+            </scan>
+            <range>
+              <min>0.060</min>
+              <max>4.095</max>
+              <resolution>0.01</resolution>
+            </range>
+            <noise>
+              <type>gaussian</type>
+              <!-- Noise parameters based on published spec for Hokuyo laser
+                  achieving "+-30mm" accuracy at range < 10m.  A mean of 0.0m and
+                  stddev of 0.01m will put 99.7% of samples within 0.03m of the true
+                  reading. -->
+              <mean>0.0</mean>
+              <stddev>0.01</stddev>
+            </noise>
+          </ray>
+      </sensor>
+    </gazebo>
+  </xacro:if>
+</xacro:macro>
+</robot>

File: urdf/stacks/circles.urdf.xacro (robot description, xacro)
@@ -18,5 +18,5 @@
         <origin xyz=" 0 0 0 " rpy="0 0 0" />
         <geometry>
-          <mesh filename="package://chris_ros_turtlebot2/models/meshes/stacks/circles/68-02403-125_Spacer.dae"/>
+          <mesh filename="file://$(find chris_ros_turtlebot2)/models/meshes/stacks/circles/68-02403-125_Spacer.dae"/>
         </geometry>
       </visual>
@@ -46,5 +46,5 @@
         <origin xyz=" 0 0 0 " rpy="0 0 0" />
         <geometry>
-          <mesh filename="package://chris_ros_turtlebot2/models/meshes/stacks/circles/68-04552-1000-RA_Turtlebot_M-F_Standoff.dae"/>
+          <mesh filename="file://$(find chris_ros_turtlebot2)/models/meshes/stacks/circles/68-04552-1000-RA_Turtlebot_M-F_Standoff.dae"/>
         </geometry>
       </visual>
@@ -74,5 +74,5 @@
         <origin xyz=" 0 0 0 " rpy="0 0 0" />
         <geometry>
-          <mesh filename="package://chris_ros_turtlebot2/models/meshes/stacks/circles/68-04552-2000-RA_Turtlebot_M-F_Standoff.dae"/>
+          <mesh filename="file://$(find chris_ros_turtlebot2)/models/meshes/stacks/circles/68-04552-2000-RA_Turtlebot_M-F_Standoff.dae"/>
         </geometry>
       </visual>
@@ -102,5 +102,5 @@
         <origin xyz=" 0 0 0 " rpy="0 0 0" />
         <geometry>
-          <mesh filename="package://chris_ros_turtlebot2/models/meshes/stacks/circles/68-02421-8000-RA_Turtlebot_F-F_Standoff.dae"/>
+          <mesh filename="file://$(find chris_ros_turtlebot2)/models/meshes/stacks/circles/68-02421-8000-RA_Turtlebot_F-F_Standoff.dae"/>
         </geometry>
       </visual>
@@ -130,5 +130,5 @@
         <origin xyz=" 0 0 0 " rpy="0 0 0" />
         <geometry>
-          <mesh filename="package://chris_ros_turtlebot2/models/meshes/stacks/circles/68-04556-RA_Kinect_Standoff_Assy.dae"/>
+          <mesh filename="file://$(find chris_ros_turtlebot2)/models/meshes/stacks/circles/68-04556-RA_Kinect_Standoff_Assy.dae"/>
         </geometry>
       </visual>
@@ -162,5 +162,5 @@
         <origin xyz=" 0 0 0 " rpy="0 0 0" />
         <geometry>
-          <mesh filename="package://chris_ros_turtlebot2/models/meshes/stacks/circles/plate_0_logo.dae"/>
+          <mesh filename="file://$(find chris_ros_turtlebot2)/models/meshes/stacks/circles/plate_0_logo.dae"/>
         </geometry>
       </visual>
@@ -192,5 +192,5 @@
         <origin xyz=" 0 0 0 " rpy="0 0 0" />
         <geometry>
-          <mesh filename="package://chris_ros_turtlebot2/models/meshes/stacks/circles/plate_1_logo.dae"/>
+          <mesh filename="file://$(find chris_ros_turtlebot2)/models/meshes/stacks/circles/plate_1_logo.dae"/>
         </geometry>
       </visual>
@@ -222,5 +222,5 @@
         <origin xyz=" 0 0 0 " rpy="0 0 0" />
         <geometry>
-          <mesh filename="package://chris_ros_turtlebot2/models/meshes/stacks/circles/plate_1_logo.dae"/>
+          <mesh filename="file://$(find chris_ros_turtlebot2)/models/meshes/stacks/circles/plate_1_logo.dae"/>
         </geometry>
       </visual>
@@ -254,5 +254,5 @@
         <origin xyz=" 0 0 0 " rpy="0 0 0" />
         <geometry>
-          <mesh filename="package://chris_ros_turtlebot2/models/meshes/stacks/circles/plate_2_logo.dae"/>
+          <mesh filename="file://$(find chris_ros_turtlebot2)/models/meshes/stacks/circles/plate_2_logo.dae"/>
         </geometry>
       </visual>

File: urdf/stacks/hexagons.urdf.xacro (robot description, xacro)
@@ -19,5 +19,5 @@
         <origin xyz="0 0 0" rpy="0 0 0"/>
         <geometry>
-          <mesh filename="package://chris_ros_turtlebot2/models/meshes/stacks/hexagons/pole_bottom.dae"/>
+          <mesh filename="file://$(find chris_ros_turtlebot2)/models/meshes/stacks/hexagons/pole_bottom.dae"/>
         </geometry>
       </visual>
@@ -47,5 +47,5 @@
         <origin xyz="0 0 0" rpy="0 ${M_PI} 0"/>
         <geometry>
-          <mesh filename="package://chris_ros_turtlebot2/models/meshes/stacks/hexagons/pole_middle.dae"/>
+          <mesh filename="file://$(find chris_ros_turtlebot2)/models/meshes/stacks/hexagons/pole_middle.dae"/>
         </geometry>
       </visual>
@@ -75,5 +75,5 @@
         <origin xyz=" 0 0 0" rpy="0 0 0"/>
         <geometry>
-          <mesh filename="package://chris_ros_turtlebot2/models/meshes/stacks/hexagons/pole_top.dae"/>
+          <mesh filename="file://$(find chris_ros_turtlebot2)/models/meshes/stacks/hexagons/pole_top.dae"/>
         </geometry>
       </visual>
@@ -103,5 +103,5 @@
         <origin xyz="0 0 0" rpy="0 0 0"/>
         <geometry>
-          <mesh filename="package://chris_ros_turtlebot2/models/meshes/stacks/hexagons/pole_kinect.dae" />
+          <mesh filename="file://$(find chris_ros_turtlebot2)/models/meshes/stacks/hexagons/pole_kinect.dae" />
         </geometry>
       </visual>
@@ -142,5 +142,5 @@
         <origin xyz="0 0 0" rpy="0 0 0"/>
         <geometry>
-          <mesh filename="package://chris_ros_turtlebot2/models/meshes/stacks/hexagons/plate_bottom.dae"/>
+          <mesh filename="file://$(find chris_ros_turtlebot2)/models/meshes/stacks/hexagons/plate_bottom.dae"/>
         </geometry>
       </visual>
@@ -172,5 +172,5 @@
         <origin xyz="0 0 0" rpy="0 0 0"/>
         <geometry>
-          <mesh filename="package://chris_ros_turtlebot2/models/meshes/stacks/hexagons/plate_middle.dae"/>
+          <mesh filename="file://$(find chris_ros_turtlebot2)/models/meshes/stacks/hexagons/plate_middle.dae"/>
         </geometry>
       </visual>
@@ -178,5 +178,5 @@
         <origin xyz="0.01364 0.0 0.0" rpy="0 0 0"/>
         <geometry>
-          <mesh filename="package://chris_ros_turtlebot2/models/meshes/stacks/hexagons/plate_simple.stl"
+          <mesh filename="file://$(find chris_ros_turtlebot2)/models/meshes/stacks/hexagons/plate_simple.stl"
                 scale="${M_SCALE} ${M_SCALE} ${M_SCALE}"/>
         </geometry>
@@ -205,5 +205,5 @@
         <origin xyz="0 0 0" rpy="0 0 0"/>
         <geometry>
-          <mesh filename="package://chris_ros_turtlebot2/models/meshes/stacks/hexagons/plate_top.dae"/>
+          <mesh filename="file://$(find chris_ros_turtlebot2)/models/meshes/stacks/hexagons/plate_top.dae"/>
         </geometry>
       </visual>
@@ -211,5 +211,5 @@
         <origin xyz="0.01364 0 0" rpy="0 0 0"/>
         <geometry>
-          <mesh filename="package://chris_ros_turtlebot2/models/meshes/stacks/hexagons/plate_simple.stl"
+          <mesh filename="file://$(find chris_ros_turtlebot2)/models/meshes/stacks/hexagons/plate_simple.stl"
                 scale="${M_SCALE} ${M_SCALE} ${M_SCALE}"/>
         </geometry>
