Commit message: debugging

File: urdf/sensors/_d435.urdf.xacro (robot description, xacro)
@@ -21,6 +21,5 @@
 <robot name="sensor_d435" xmlns:xacro="http://ros.org/wiki/xacro">
   <!-- Includes -->
-  <xacro:include filename="$(find chris_ros_turtlebot2)/urdf/sensors/_materials.urdf.xacro" />
-  <xacro:include filename="$(find chris_ros_turtlebot2)/urdf/sensors/_usb_plug.urdf.xacro" />
+  <xacro:include filename="$(find chris_ros_turtlebot2)/urdf/_d435.gazebo.xacro" />
   <xacro:macro name="sensor_d435" params="parent *origin name:=camera use_nominal_extrinsics:=false add_plug:=false use_mesh:=true">
     <xacro:property name="M_PI" value="3.1415926535897931" />

File: urdf/sensors/_d435i.urdf.xacro (robot description, xacro)
@@ -22,8 +22,9 @@
   <xacro:include filename="$(find chris_ros_turtlebot2)/urdf/sensors/_d435.urdf.xacro"/>
   <xacro:include filename="$(find chris_ros_turtlebot2)/urdf/sensors/_d435i_imu_modules.urdf.xacro"/>
-  <xacro:macro name="sensor_d435i" params="parent *origin name:=camera use_nominal_extrinsics:=false">
-    <xacro:sensor_d435 parent="${parent}" name="${name}" use_nominal_extrinsics="${use_nominal_extrinsics}">
+  <xacro:macro name="sensor_d435i" params="parent name:=camera use_nominal_extrinsics:=false">
+  <!-- <xacro:macro name="sensor_d435i" params="parent *origin name:=camera use_nominal_extrinsics:=false"> -->
+    <!-- <xacro:sensor_d435 parent="${parent}" name="${name}" use_nominal_extrinsics="${use_nominal_extrinsics}">
       <xacro:insert_block name="origin" />
-    </xacro:sensor_d435>
+    </xacro:sensor_d435> -->
     <xacro:d435i_imu_modules name="${name}" use_nominal_extrinsics="${use_nominal_extrinsics}"/>
   </xacro:macro>

Commit message: Restore commented block, add origin

File: urdf/sensors/_d435.urdf.xacro (robot description, xacro)
@@ -22,4 +22,6 @@
   <!-- Includes -->
   <xacro:include filename="$(find chris_ros_turtlebot2)/urdf/_d435.gazebo.xacro" />
+  <xacro:include filename="$(find chris_ros_turtlebot2)/urdf/sensors/_materials.urdf.xacro"/>
+  <xacro:include filename="$(find chris_ros_turtlebot2)/urdf/sensors/_usb_plug.urdf.xacro"/>
   <xacro:macro name="sensor_d435" params="parent *origin name:=camera use_nominal_extrinsics:=false add_plug:=false use_mesh:=true">
     <xacro:property name="M_PI" value="3.1415926535897931" />

File: urdf/sensors/_d435i.urdf.xacro (robot description, xacro)
@@ -22,9 +22,8 @@
   <xacro:include filename="$(find chris_ros_turtlebot2)/urdf/sensors/_d435.urdf.xacro"/>
   <xacro:include filename="$(find chris_ros_turtlebot2)/urdf/sensors/_d435i_imu_modules.urdf.xacro"/>
-  <xacro:macro name="sensor_d435i" params="parent name:=camera use_nominal_extrinsics:=false">
-  <!-- <xacro:macro name="sensor_d435i" params="parent *origin name:=camera use_nominal_extrinsics:=false"> -->
-    <!-- <xacro:sensor_d435 parent="${parent}" name="${name}" use_nominal_extrinsics="${use_nominal_extrinsics}">
+  <xacro:macro name="sensor_d435i" params="parent *origin name:=camera use_nominal_extrinsics:=false">
+    <xacro:sensor_d435 parent="${parent}" name="${name}" use_nominal_extrinsics="${use_nominal_extrinsics}">
       <xacro:insert_block name="origin" />
-    </xacro:sensor_d435> -->
+    </xacro:sensor_d435>
     <xacro:d435i_imu_modules name="${name}" use_nominal_extrinsics="${use_nominal_extrinsics}"/>
   </xacro:macro>
