Commit message: Add the missing block value

File: robots/kobuki_hexagons_d435if_hokuyo.urdf.xacro (robot description, xacro)
@@ -13,5 +13,7 @@
   <xacro:kobuki/>
   <xacro:stack_hexagons parent="base_link"/>
-  <xacro:sensor_d435i   parent="base_link"/>
+  <xacro:sensor_d435i   parent="base_link">
+    <origin xyz="0.095 0 0.37" rpy="0 0 0" />
+  </xacro:sensor_d435i>
   <joint name="hokuyo_base_joint" type="fixed">
     <axis xyz="0 0 1" />
